File: pcb/myFarm.kicad_pcb (KiCad board)
At the start: 2 copper layers, 63.5 x 52.1 mm, 10 parts, among them J0 Conn_01x02, J1 LED, J2 SENSOR, J3 SW_LED, J4 RELAY, J5 POWER DRIVE, J6 JUMPER, J7 SW_LED, U1 WeMos_D1_mini, U2 MCP23017_MODULE

Commit message: update pcb
Parts:
- added J10: GENERAL, Connector_PinHeader_2.54mm:PinHeader_1x06_P2.54mm_Vertical, F.Cu at (69.8, 72.4)
- added J11: RXTX, Connector_PinHeader_2.54mm:PinHeader_1x02_P2.54mm_Vertical, F.Cu at (104.1, 82.5)
- added J12: VALVE OUT, Connector_PinHeader_2.54mm:PinHeader_1x02_P2.54mm_Vertical, F.Cu at (104.1, 94.0)
- added J13: VALVE OUT, Connector_PinHeader_2.54mm:PinHeader_1x02_P2.54mm_Vertical, F.Cu at (111.8, 94.0)
- added J14: VALVE OUT, Connector_PinHeader_2.54mm:PinHeader_1x02_P2.54mm_Vertical, F.Cu at (119.4, 94.0)
- added J8: Reset, Connector_PinHeader_2.54mm:PinHeader_1x02_P2.54mm_Vertical, F.Cu at (91.4, 95.2)
- added J9: VAVLE IN, Connector_PinHeader_2.54mm:PinHeader_1x02_P2.54mm_Vertical, F.Cu at (96.5, 94.0)
- added U3: DS1832S+, Package_DIP:DIP-8_W10.16mm, B.Cu at (91.4, 78.7)
- J0: value Conn_01x02 -> POWER
- J7: value SW_LED -> SUPPLY
- moved J6 6.35 mm to (85.1, 69.8), turned to 90 degrees
- moved J0 1.80 mm to (111.8, 50.8)
- moved U2 1.80 mm to (102.9, 62.2)
- moved J4 1.80 mm to (118.1, 62.2)
- moved J7 1.80 mm to (109.2, 57.1)
- moved J1 1.80 mm to (77.5, 55.9)
- moved J2 1.80 mm to (69.8, 81.3)
- moved J3 1.80 mm to (86.4, 55.9)
- moved J5 1.80 mm to (118.1, 76.2)
- moved U1 1.80 mm to (77.5, 86.4)
Connections:
- U1 pad 1: (no net) -> Net-(U1-Pad1)
- U1 pad 15: (no net) -> Net-(J11-Pad2)
- U1 pad 16: (no net) -> Net-(J11-Pad1)
- U1 pad 2: (no net) -> Net-(J10-Pad1)
- U1 pad 3: (no net) -> Net-(J10-Pad2)
- U1 pad 5: (no net) -> Net-(U1-Pad5)
- U1 pad 6: (no net) -> Net-(J10-Pad3)
- U1 pad 7: (no net) -> Net-(J10-Pad4)
- U2 pad 5: (no net) -> Net-(J9-Pad1)
- U2 pad 6: (no net) -> Net-(J12-Pad1)
- U2 pad 7: (no net) -> Net-(J13-Pad1)
- U2 pad 8: (no net) -> Net-(J14-Pad1)
Routing:
- net GNDREF: track 146.4 -> 191.7 mm
- net Net-(J6-Pad3): track 69.3 -> 30.1 mm
- net Net-(J8-Pad2): track 0.00 -> 18.3 mm
- net Net-(J10-Pad1): track 0.00 -> 17.6 mm
- net Net-(J10-Pad2): track 0.00 -> 16.8 mm
- net Net-(U1-Pad5): track 0.00 -> 12.5 mm
- net Net-(J10-Pad3): track 0.00 -> 11.1 mm
- net Net-(J6-Pad2): track 20.4 -> 9.42 mm
- net Net-(J9-Pad1): track 0.00 -> 10.8 mm
- net Net-(J10-Pad4): track 0.00 -> 10.3 mm
- net Net-(J12-Pad1): track 0.00 -> 7.18 mm
- net Net-(J1-Pad1): track 145.0 -> 150.5 mm
- net Net-(U1-Pad1): track 0.00 -> 4.86 mm
- net Net-(J13-Pad1): track 0.00 -> 3.59 mm
- net Net-(J1-Pad2): track 37.8 -> 38.5 mm

Commit message: update pcb.
Parts:
- added J15: LED, Connector_PinHeader_2.54mm:PinHeader_1x02_P2.54mm_Vertical, B.Cu at (91.4, 94.0)
- J11: moved to B.Cu
- moved J6 6.35 mm to (85.1, 76.2), turned to 180 degrees
- moved J8 4.02 mm to (87.6, 94.0)
- moved J11 1.27 mm to (104.1, 83.8)
Connections:
- U1 pad 11: (no net) -> Net-(J15-Pad2)
Routing:
- net GNDREF: track 191.7 -> 224.5 mm
- net Net-(J9-Pad1): track 10.8 -> 24.0 mm
- net Net-(J14-Pad1): track 0.00 -> 12.3 mm
- net Net-(J13-Pad1): track 3.59 -> 12.3 mm
- net Net-(J12-Pad1): track 7.18 -> 12.3 mm
- net Net-(J1-Pad1): track 150.5 -> 146.4 mm
- net Net-(J11-Pad2): track 0.00 -> 3.81 mm
- net Net-(J11-Pad1): track 0.00 -> 3.81 mm
- net Net-(J6-Pad2): track 9.42 -> 8.89 mm

Commit message: update pcb.
Parts:
- J15: moved to F.Cu
- moved J8 17.8 mm to (69.8, 94.0), turned to 90 degrees
- moved J11 2.54 mm to (104.1, 86.4), turned to 0 degrees
- moved J15 2.54 mm to (88.9, 94.0), turned to 90 degrees
Routing:
- net Net-(J15-Pad2): track 0.00 -> 26.4 mm
- net GNDREF: track 224.5 -> 243.7 mm
- net Net-(J8-Pad2): track 18.6 -> 29.1 mm
- net Net-(J6-Pad3): track 30.1 -> 37.0 mm
- net Net-(U1-Pad5): track 12.5 -> 11.7 mm

Commit message: update pcb.
Parts:
- J15: value LED -> SELECTOR
- J5: footprint Connector_PinHeader_2.54mm:PinHeader_1x06_P2.54mm_Vertical -> Connector_PinHeader_2.54mm:PinHeader_1x08_P2.54mm_Vertical
- moved J14 10.2 mm to (109.2, 94.0), turned to 0 degrees
- moved J13 7.62 mm to (104.1, 94.0), turned to 0 degrees
- moved J12 5.08 mm to (99.1, 94.0), turned to 0 degrees
- moved J15 4.58 mm to (85.1, 96.5), turned to 180 degrees
- moved J9 2.54 mm to (94.0, 94.0), turned to 0 degrees
Routing:
- net Net-(J1-Pad1): track 146.4 -> 181.3 mm
- net GNDREF: track 243.7 -> 260.2 mm
- net Net-(J14-Pad1): track 12.3 -> 5.08 mm
- net Net-(J15-Pad2): track 26.4 -> 32.0 mm
- net Net-(J12-Pad1): track 12.3 -> 15.2 mm
- net Net-(J13-Pad1): track 12.3 -> 9.72 mm

Commit message: update pcb
Parts:
- J0: footprint Connector_PinHeader_2.54mm:PinHeader_1x02_P2.54mm_Horizontal -> Connector_JST:JST_XH_B2B-XH-A_1x02_P2.50mm_Vertical
- J1, J11, J12, J13, J14, J15, J8, J9: footprint Connector_PinHeader_2.54mm:PinHeader_1x02_P2.54mm_Vertical -> Connector_JST:JST_XH_B2B-XH-A_1x02_P2.50mm_Vertical
- J10: footprint Connector_PinHeader_2.54mm:PinHeader_1x06_P2.54mm_Vertical -> Connector_JST:JST_XH_B6B-XH-A_1x06_P2.50mm_Vertical
- J2: footprint Connector_PinHeader_2.54mm:PinHeader_1x03_P2.54mm_Vertical -> Connector_JST:JST_XH_B3B-XH-A_1x03_P2.50mm_Vertical
- J3, J4: footprint Connector_PinHeader_2.54mm:PinHeader_1x04_P2.54mm_Vertical -> Connector_JST:JST_XH_B4B-XH-A_1x04_P2.50mm_Vertical
- J5: footprint Connector_PinHeader_2.54mm:PinHeader_1x08_P2.54mm_Vertical -> Connector_JST:JST_XH_B8B-XH-A_1x08_P2.50mm_Vertical
- J7: footprint Module:POWER_SUPPLY_MODULE -> Connector_JST:JST_XH_B4B-XH-A_1x04_P2.50mm_Vertical
- U3: footprint Package_DIP:DIP-8_W10.16mm -> Package_DIP:DIP-8_W7.62mm_Socket
- moved J15 10.5 mm to (74.9, 94.0), turned to 0 degrees
- moved J9 10.2 mm to (83.8, 94.0)
- moved J0 8.03 mm to (119.4, 53.3), turned to 270 degrees
- moved J6 7.73 mm to (86.4, 68.6), turned to 0 degrees
- moved U2 6.48 mm to (104.1, 55.9)
- moved J12 6.35 mm to (92.7, 94.0)
- moved J7 4.02 mm to (110.5, 53.3), turned to 180 degrees
- moved J3 3.59 mm to (88.9, 53.3), turned to 0 degrees
- moved J10 2.84 mm to (68.6, 69.8), turned to 90 degrees
- moved J8 2.84 mm to (68.6, 91.4)
- moved J13 2.54 mm to (101.6, 94.0)
- moved J1 2.54 mm to (77.5, 53.3), turned to 0 degrees
- moved J11 1.27 mm to (105.4, 86.4), turned to 90 degrees
- moved J14 1.27 mm to (110.5, 94.0)
- moved J2 1.27 mm to (68.6, 81.3), turned to 90 degrees
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Routing:
- net GNDREF: track 260.2 -> 0.00 mm
- net Net-(J6-Pad3): track 37.0 -> 15.0 mm
- net Net-(J9-Pad1): track 23.5 -> 40.8 mm
- net Net-(J12-Pad1): track 15.2 -> 32.1 mm
- net Net-(J13-Pad1): track 9.72 -> 20.6 mm
- net Net-(J0-Pad1): track 8.89 -> 17.9 mm
- net Net-(J3-Pad3): track 38.1 -> 30.2 mm
- net Net-(J15-Pad2): track 32.0 -> 38.7 mm
- net Net-(J14-Pad1): track 5.08 -> 11.4 mm
- net Net-(J3-Pad2): track 40.2 -> 34.5 mm
- net Net-(J5-Pad6): track 6.35 -> 11.9 mm
- net Net-(J10-Pad4): track 10.3 -> 15.6 mm
- net Net-(J10-Pad3): track 11.1 -> 16.2 mm
- net Net-(J5-Pad5): track 6.35 -> 11.1 mm
- net Net-(J1-Pad1): track 181.3 -> 177.1 mm
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- added copper zone on B.Cu, net GNDREF
- added copper zone on F.Cu, net GNDREF
