File: pcb/myFarm.kicad_pcb (KiCad board)
At the start: 2 copper layers, 63.5 x 52.1 mm, 19 parts, among them J0 POWER, J1 LED, J10 GENERAL, J11 RXTX, J12 VALVE OUT, J13 VALVE OUT, J14 VALVE OUT, J15 SELECTOR, J2 SENSOR, J3 SW_LED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

Commit message: update pcb board.
Parts:
- added J16: Conn_01x02, Connector_JST:JST_XH_B4B-XH-A_1x04_P2.50mm_Vertical, F.Cu at (82.5, 68.6)
- added J17: Conn_01x02, Connector_JST:JST_XH_B4B-XH-A_1x04_P2.50mm_Vertical, F.Cu at (88.9, 68.6)
- J11: footprint Connector_JST:JST_XH_B2B-XH-A_1x02_P2.50mm_Vertical -> Connector_JST:JST_XH_B4B-XH-A_1x04_P2.50mm_Vertical
- moved J6 6.35 mm to (82.5, 73.7), turned to 90 degrees
- moved J11 2.54 mm to (105.4, 88.9)
Connections:
- J11 pad 1: Net-(J11-Pad1) -> Net-(J1-Pad1)
- U1 pad 15: Net-(J11-Pad2) -> Net-(J11-Pad3)
- U1 pad 16: Net-(J11-Pad1) -> Net-(J11-Pad2)
Routing:
- net Net-(J16-Pad2): track 6.66 -> 29.4 mm
- net Net-(J16-Pad3): track 6.66 -> 22.9 mm
- net Net-(J6-Pad3): track 15.0 -> 0.00 mm
- net Net-(J6-Pad2): track 11.2 -> 0.00 mm
- net Net-(J11-Pad3): track 0.00 -> 5.10 mm
- net Net-(J11-Pad1): track 5.08 -> 0.00 mm
- net Net-(J1-Pad1): track 177.1 -> 179.6 mm

Commit message: update pcb
Parts:
- added J18: LED, Connector_Wire:SolderWirePad_1x02_P7.62mm_Drill2.5mm, F.Cu at (133.3, 92.7)
- added J19: POWER, Connector_Wire:SolderWirePad_1x02_P7.62mm_Drill2.5mm, F.Cu at (133.3, 53.3)
- added U4: TA6586, Package_DIP:DIP-8_W7.62mm_Socket, F.Cu at (129.5, 68.6)
Routing:
- net Net-(J0-Pad1): track 17.9 -> 57.0 mm
- net Net-(J18-Pad1): track 0.00 -> 32.4 mm
- net Net-(J18-Pad2): track 0.00 -> 21.6 mm
- net Net-(J1-Pad1): track 179.6 -> 195.4 mm
- net Net-(J6-Pad2): track 0.00 -> 14.3 mm
- net Net-(J6-Pad3): track 0.00 -> 13.8 mm
- net Net-(J4-Pad3): track 6.38 -> 18.2 mm
- net Net-(J4-Pad2): track 6.37 -> 18.1 mm
- net Net-(J16-Pad3): track 22.9 -> 29.3 mm
Other:
- board size 63.5 x 52.1 mm -> 82.6 x 52.1 mm

Commit message: new version pcb
Parts:
- removed J15: SELECTOR, Connector_JST:JST_XH_B2B-XH-A_1x02_P2.50mm_Vertical
- J10: value GENERAL -> SR04; footprint Connector_JST:JST_XH_B6B-XH-A_1x06_P2.50mm_Vertical -> Connector_JST:JST_XH_B4B-XH-A_1x04_P2.50mm_Vertical
- J11: moved to F.Cu
- J12: value VALVE OUT -> VALVE IN
- J16, J17: value Conn_01x02 -> I2C
- J18: value LED -> PUMP
- J5: value POWER DRIVE -> configuration; footprint Connector_JST:JST_XH_B8B-XH-A_1x08_P2.50mm_Vertical -> Connector_PinHeader_2.00mm:PinHeader_2x04_P2.00mm_Vertical; moved to B.Cu
- J7: value SUPPLY -> SUPPLY 3.3
- moved J9 40.7 mm to (124.5, 96.5), turned to 180 degrees
- moved J2 38.7 mm to (104.1, 96.5), turned to 180 degrees
- moved J12 32.2 mm to (124.5, 88.9), turned to 180 degrees
- moved J3 31.5 mm to (68.6, 77.5), turned to 90 degrees
- moved J10 27.7 mm to (76.2, 96.5), turned to 180 degrees
- moved J16 19.4 mm to (72.4, 52.1), turned to 0 degrees
- moved J17 16.6 mm to (87.6, 52.1), turned to 0 degrees
- moved J11 15.9 mm to (91.4, 96.5), turned to 180 degrees
- moved J5 14.4 mm to (106.0, 81.3), turned to 0 degrees
- moved J1 13.5 mm to (68.6, 63.5), turned to 90 degrees
- moved J13 13.0 mm to (114.3, 96.5), turned to 180 degrees
- moved J19 7.62 mm to (133.3, 61.0), turned to 90 degrees
- moved J14 6.35 mm to (114.3, 88.9), turned to 180 degrees
- moved U1 4.02 mm to (78.7, 82.5)
- moved J8 3.81 mm to (68.6, 87.6)
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Connections:
- net Net-(J0-Pad1) renamed +12V
- J1 pad 1: Net-(J1-Pad1) -> +3V3
- J10 pad 1: Net-(J10-Pad1) -> GNDREF
- J10 pad 4: Net-(J10-Pad4) -> +3V3
- J11 pad 1: Net-(J1-Pad1) -> +3V3
- J16 pad 1: Net-(J1-Pad1) -> +3V3
- J17 pad 1: Net-(J1-Pad1) -> +3V3
- J2 pad 1: Net-(J1-Pad1) -> +3V3
- J3 pad 1: Net-(J1-Pad1) -> +3V3
- J4 pad 1: Net-(J1-Pad1) -> +3V3
- J5 pad 1: Net-(J5-Pad1) -> GNDREF
- J5 pad 3: Net-(J5-Pad3) -> GNDREF
- J5 pad 5: Net-(J5-Pad5) -> GNDREF
- J5 pad 7: Net-(J1-Pad1) -> GNDREF
- J5 pad 8: GNDREF -> Net-(J5-Pad8)
- J6 pad 1: Net-(J1-Pad1) -> +3V3
- J7 pad 1: Net-(J1-Pad1) -> +3V3
- U1 pad 11: Net-(J15-Pad2) -> Net-(J10-Pad3)
- U1 pad 12: Net-(J6-Pad3) -> Net-(J10-Pad2)
- U1 pad 2: Net-(J10-Pad1) -> (no net)
- U1 pad 3: Net-(J10-Pad2) -> Net-(U1-Pad3)
- U1 pad 5: Net-(U1-Pad5) -> (no net)
- U1 pad 6: Net-(J10-Pad3) -> (no net)
- U1 pad 7: Net-(J10-Pad4) -> Net-(J6-Pad3)
- U1 pad 8: Net-(J1-Pad1) -> +3V3
- U2 pad 23: Net-(J5-Pad1) -> Net-(J9-Pad1)
- U2 pad 24: Net-(J5-Pad2) -> Net-(J12-Pad1)
- U2 pad 25: Net-(J5-Pad3) -> Net-(J13-Pad1)
- U2 pad 26: Net-(J5-Pad4) -> Net-(J14-Pad1)
- U2 pad 27: Net-(J5-Pad5) -> (no net)
- U2 pad 28: Net-(J5-Pad6) -> (no net)
- U2 pad 29: Net-(J1-Pad1) -> +3V3
- U2 pad 5: Net-(J9-Pad1) -> Net-(J5-Pad8)
- U2 pad 6: Net-(J12-Pad1) -> Net-(J5-Pad6)
- U2 pad 7: Net-(J13-Pad1) -> Net-(J5-Pad4)
- U2 pad 8: Net-(J14-Pad1) -> Net-(J5-Pad2)
- U2 pad 9: Net-(J1-Pad1) -> +3V3
- U3 pad 2: Net-(J1-Pad1) -> +3V3
- U3 pad 7: Net-(U1-Pad5) -> Net-(U1-Pad3)
- U3 pad 8: Net-(J1-Pad1) -> +3V3
Routing:
- net +3V3: track 0.00 -> 206.2 mm
- net Net-(J1-Pad1): track 195.4 -> 0.00 mm
- net Net-(J15-Pad2): track 38.7 -> 0.00 mm
- net Net-(J3-Pad3): track 30.2 -> 66.5 mm
- net Net-(J10-Pad3): track 16.2 -> 51.8 mm, vias 0 -> 1
- net Net-(J2-Pad2): track 8.91 -> 44.2 mm, vias 0 -> 1
- net Net-(J3-Pad2): track 34.5 -> 67.5 mm
- net Net-(J10-Pad2): track 19.9 -> 47.5 mm, vias 0 -> 1
- net Net-(J11-Pad3): track 5.10 -> 29.5 mm
- net Net-(J16-Pad2): track 29.4 -> 52.9 mm
- net Net-(J16-Pad3): track 29.3 -> 50.8 mm
- net Net-(J10-Pad1): track 20.5 -> 0.00 mm
- net Net-(J11-Pad2): track 5.08 -> 24.4 mm
- net Net-(J1-Pad2): track 35.3 -> 52.5 mm
- net Net-(J10-Pad4): track 15.6 -> 0.00 mm
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Other:
- net class 3.3v added: clearance 0.2, trace_width 1, via_dia 0.8, via_drill 0.4
