File: pcb/myFarm.sch (KiCad schematic (older format))
At the start: 21 parts, among them J0 POWER, J1 LED, J10 GENERAL, J11 RXTX, J12 VALVE OUT, J13 VALVE OUT, J14 VALVE OUT, J15 SELECTOR, J16 Conn_01x02, J17 Conn_01x02, J2 SENSOR, J3 SW_LED, J4 RELAY, J5 POWER DRIVE, J6 JUMPER, J7 SUPPLY, J8 Reset, J9 VAVLE IN, U1 WeMos_D1_mini, U2 MCP23017_MODULE, U3 DS1832S+

Commit message: update pcb
Parts:
- added J18: LED, Connector_Wire:SolderWirePad_1x02_P7.62mm_Drill2.5mm, symbol Connector_Generic:Conn_01x02
- added J19: POWER, Connector_Wire:SolderWirePad_1x02_P7.62mm_Drill2.5mm, symbol Connector_Generic:Conn_01x02
- added U4: TA6586, Package_DIP:DIP-8_W7.62mm_Socket, symbol TA6586:TA6586
Connections:
- net GNDREF: now also J19.2 (Pin_2), U4.3 (Gnd)
- net at J4.2 (Pin_2), U2.21 (A0): now also U4.1 (I1)
- net at J4.3 (Pin_3), U2.22 (A1): now also U4.2 (I2)
- net at J0.1 (Pin_1), J7.3 (Pin_3): now also J19.1 (Pin_1), U4.4 (Vcc)
- new net: J18.1 (Pin_1), U4.5 (OUTA1), U4.6 (OUTA2)
- new net: J18.2 (Pin_2), U4.7 (OUTB1), U4.8 (OUTB2)
Changed lines of the file:
@@
 Wire Wire Line
 	8650 3400 9050 3400
-Wire Wire Line
-	9050 3700 8400 3700
-Connection ~ 8400 3700
 $Comp
 L Connector_Generic:Conn_01x04 J4
@@
 Connection ~ 5550 2550
 Wire Wire Line
-	8000 3600 8350 3600
-Wire Wire Line
-	8350 3600 8350 3500
-Wire Wire Line
-	8350 3500 9050 3500
-Wire Wire Line
 	8000 3500 8250 3500
 Wire Wire Line
@@
 	3300 1650 3300 1700
 Wire Wire Line
-	3200 1850 3200 1650
+	3200 1850 3200 1800
 $Comp
 L Connector_Generic:Conn_01x04 J7
@@
 Connection ~ 4250 2550
 Wire Wire Line
-	3300 1700 2300 1700
+	3300 1700 2750 1700
 Wire Wire Line
 	2300 3950 2550 3950
@@
 Wire Wire Line
 	6950 1800 6950 2200
-Wire Wire Line
-	6950 2200 8400 2200
 Wire Wire Line
 	5550 2550 6400 2550
@@
 Wire Wire Line
 	8650 2450 8650 3400
-Wire Wire Line
-	8400 2200 8400 3700
 $Comp
 L Connector_Generic:Conn_01x03 J2
@@
 	8300 2000 8300 1800
 Wire Wire Line
-	8150 2000 8150 3900
-Wire Wire Line
 	8200 2100 8600 2100
 Wire Wire Line
@@
 Wire Wire Line
 	8700 1950 8700 2200
-Wire Wire Line
-	8700 2200 8400 2200
-Connection ~ 8400 2200
 Wire Wire Line
 	8700 1800 8700 1950
@@
 Wire Wire Line
 	4850 2450 5350 2450
+$Comp
+L TA6586:TA6586 U4
+U 1 1 5E2B7543
+P 10050 3000
+F 0 "U4" H 10050 3681 50  0000 C CNN
+F 1 "TA6586" H 10050 3590 50  0000 C CNN
+F 2 "Package_DIP:DIP-8_W7.62mm_Socket" H 10050 3300 50  0001 C CNN
+F 3 "" H 10050 3300 50  0001 C CNN
+	1    10050 3000
+	1    0    0    -1
+$EndComp
+Wire Wire Line
+	8300 4000 8300 2800
+Wire Wire Line
+	8300 2800 9700 2800
+Connection ~ 8300 4000
+Connection ~ 8400 2200
+Wire Wire Line
+	6950 2200 8400 2200
+Connection ~ 8400 3700
+Wire Wire Line
+	9050 3700 8400 3700
+Wire Wire Line
+	8700 2200 8400 2200
+Wire Wire Line
+	8150 2000 8150 3900
+Wire Wire Line
+	8400 2200 8400 3700
+Wire Wire Line
+	8600 3600 8600 3500
+Wire Wire Line
+	8000 3600 8600 3600
+Wire Wire Line
+	8600 3500 9050 3500
+Wire Wire Line
+	8350 4100 8350 3250
+Wire Wire Line
+	8350 3250 9700 3250
+Connection ~ 8350 4100
+Wire Wire Line
+	10050 5700 10050 3550
+Wire Wire Line
+	8400 5700 10050 5700
+Connection ~ 8400 5700
+Wire Wire Line
+	8650 2450 8650 2300
+$Comp
+L Connector_Generic:Conn_01x02 J18
+U 1 1 5E375647
+P 10850 2950
+F 0 "J18" H 10930 2942 50  0000 L CNN
+F 1 "LED" H 10930 2851 50  0000 L CNN
+F 2 "Connector_Wire:SolderWirePad_1x02_P7.62mm_Drill2.5mm" H 10850 2950 50  0001 C CNN
+F 3 "~" H 10850 2950 50  0001 C CNN
+	1    10850 2950
+	1    0    0    -1
+$EndComp
+Wire Wire Line
+	10650 3050 10650 3150
+Wire Wire Line
+	10650 3250 10400 3250
+Wire Wire Line
+	10400 3150 10650 3150
+Connection ~ 10650 3150
+Wire Wire Line
+	10650 3150 10650 3250
+Wire Wire Line
+	10400 2800 10650 2800
+Wire Wire Line
+	10650 2800 10650 2900
+Wire Wire Line
+	10400 2900 10650 2900
+Connection ~ 10650 2900
+Wire Wire Line
+	10650 2900 10650 2950
+$Comp
+L Connector_Generic:Conn_01x02 J19
+U 1 1 5E3BCE7F
+P 2650 1450
+F 0 "J19" V 2614 1262 50  0000 R CNN
+F 1 "POWER" V 2523 1262 50  0000 R CNN
+F 2 "Connector_Wire:SolderWirePad_1x02_P7.62mm_Drill2.5mm" H 2650 1450 50  0001 C CNN
+F 3 "~" H 2650 1450 50  0001 C CNN
+	1    2650 1450
+	0    -1   -1   0
+$EndComp
+Wire Wire Line
+	2650 1650 2650 1800
+Wire Wire Line
+	2650 1800 3200 1800
+Connection ~ 3200 1800
+Wire Wire Line
+	3200 1800 3200 1650
+Wire Wire Line
+	2750 1650 2750 1700
+Connection ~ 2750 1700
+Wire Wire Line
+	2750 1700 2300 1700
+Wire Wire Line
+	2650 1800 2450 1800
+Wire Wire Line
+	2450 1800 2450 800
+Wire Wire Line
+	2450 800  10050 800
+Wire Wire Line
+	10050 800  10050 2500
+Connection ~ 2650 1800
 $EndSCHEMATC

Commit message: new version pcb
Parts:
- removed J10: GENERAL, Connector_JST:JST_XH_B6B-XH-A_1x06_P2.50mm_Vertical, symbol Connector_Generic:Conn_01x06
- removed J15: SELECTOR, Connector_JST:JST_XH_B2B-XH-A_1x02_P2.50mm_Vertical, symbol Connector_Generic:Conn_01x02
- removed J5: POWER DRIVE, Connector_JST:JST_XH_B8B-XH-A_1x08_P2.50mm_Vertical, symbol Connector_Generic:Conn_01x08
- added J10: SR04, Connector_JST:JST_XH_B4B-XH-A_1x04_P2.50mm_Vertical, symbol Connector_Generic:Conn_01x04
- added J5: configuration, Connector_PinHeader_2.00mm:PinHeader_2x04_P2.00mm_Vertical, symbol Connector_Generic:Conn_02x04_Odd_Even
- J12: value VALVE OUT -> VALVE IN
- J16, J17: value Conn_01x02 -> I2C
- J18: value LED -> PUMP
- J7: value SUPPLY -> SUPPLY 3.3
Connections:
- net GNDREF: now also J10.1 (Pin_1), J5.1 (Pin_1), J5.3 (Pin_3), J5.5 (Pin_5), J5.7 (Pin_7)
- net at U1.11 (D4): now also J10.3 (Pin_3)
- net at U1.12 (D3): now also J10.2 (Pin_2); no longer J6.3 (Pin_3)
- net at U1.3 (D0): now also U3.7 (~ST~)
- net at U1.5 (MISO/D6): no longer U3.7 (~ST~)
- net at U1.7 (CS/D8): now also J6.3 (Pin_3)
- net +3V3: now reaches J1.1 (Pin_1), J11.1 (Pin_1), J16.1 (Pin_1), J17.1 (Pin_1), J2.1 (Pin_1), J3.1 (Pin_1), J4.1 (Pin_1), J6.1 (Pin_1), J7.1 (Pin_1), U1.8 (3V3), U2.29 (VCC), U2.9 (VCC), U3.2 (TD), U3.8 (VCC)
- net +3V3: now also J10.4 (Pin_4)
- net +5V: now reaches U1.9 (5V)
- net at U2.23 (A2): now also J9.1 (Pin_1)
- net at U2.24 (A3): now also J12.1 (Pin_1)
- net at U2.25 (A4): now also J13.1 (Pin_1)
- net at U2.26 (A5): now also J14.1 (Pin_1)
- net at U2.5 (B4): now also J5.8 (Pin_8); no longer J9.1 (Pin_1)
- net at U2.6 (B5): now also J5.6 (Pin_6); no longer J12.1 (Pin_1)
- net at U2.7 (B6): now also J5.4 (Pin_4); no longer J13.1 (Pin_1)
- net at U2.8 (B7): now also J5.2 (Pin_2); no longer J14.1 (Pin_1)
- net +12V: now reaches J0.1 (Pin_1), J19.1 (Pin_1), J7.3 (Pin_3), U4.4 (Vcc)
Other:
- moved on the sheet: J12, J13, J14, J9
